Commit message: added gps link and sensor

File: src/turtlebot3/turtlebot3_description/urdf/turtlebot3_waffle.urdf (robot description, URDF)
Before this commit: robot turtlebot3_waffle, 13 links, 12 joints
Links:
- added link gps_link
Joints:
- added joint gps_joint: type fixed, parent base_link, child gps_link, origin xyz=0.0 0 0.068 rpy=0 0 0
- joint imu_joint: origin xyz=0.0 0 0.068 rpy=0 0 0 -> xyz=-0.032 0 0.068 rpy=0 0 0

Commit message: removed all the useless sensors

File: src/turtlebot3/turtlebot3_description/urdf/turtlebot3_waffle.urdf (robot description, URDF)
Before this commit: robot turtlebot3_waffle, 14 links, 13 joints
Links:
- removed link base_scan
- removed link camera_depth_frame
- removed link camera_depth_optical_frame
- removed link camera_link
- removed link camera_rgb_frame
- removed link camera_rgb_optical_frame
Joints:
- removed joint camera_depth_joint
- removed joint camera_depth_optical_joint
- removed joint camera_joint
- removed joint camera_rgb_joint
- removed joint camera_rgb_optical_joint
- removed joint scan_joint
